File: ElectricalProject/ArduinoIHM.kicad_sch (KiCad schematic)
At the start: 76 parts, among them J1 PWR-CONNECTORS, J10 AN0, J11 AN1, J12 AN2, J13 AN3, J14 PWR, J15 DAC0_out, J16 DAC1, J17 DAC1_out, J18 Can0, J19 Can1, J2 PF 0 - 7, J20 RS485, J21 PWM0, J22 PWM1, J23 PWM2, J24 D-J3, J25 D-J4, J26 D-J2, J27 D-J1, J28 COMM, J29 Conn_01x10, J3 PK 8-15, J30 OrientationDet, J31 ServoSig, J32 VccLine, J33 GndLine, J34 DCMotorOut, J4 Conn_01x08, J5 Conn_01x08, J6 PWM, J7 DigitalIO, J8 external_PWR, J9 DAC0, Q1 BC547, SW1 RotaryEncoder_Switch, SW2 RotaryEncoder_Switch, SW3 RotaryEncoder_Switch, SW4 SW_Push, SW5 SW_Push, SW6 SW_Push, SW7 SW_Push, U1 LM741, U2 74LS373, U3 74LS373, U4 74LS373

Commit message: Electrical project update - fix page size
Parts:
- removed J10: AN0, symbol Connector_Generic_MountingPin:Conn_01x02_MountingPin
- removed J11: AN1, symbol Connector_Generic_MountingPin:Conn_01x02_MountingPin
- removed J12: AN2, symbol Connector_Generic_MountingPin:Conn_01x02_MountingPin
- removed J13: AN3, symbol Connector_Generic_MountingPin:Conn_01x02_MountingPin
- removed NEG_BMX_INOUT: POS_BMS_INOUT, symbol Connector_Generic_MountingPin:Conn_01x02_MountingPin
- added J10: AN1, Connector_PinHeader_2.54mm:PinHeader_1x02_P2.54mm_Vertical, symbol Connector_Generic:Conn_01x02
- added J11: AN2, Connector_PinHeader_2.54mm:PinHeader_1x02_P2.54mm_Vertical, symbol Connector_Generic:Conn_01x02
- added J12: AN3, Connector_PinHeader_2.54mm:PinHeader_1x02_P2.54mm_Vertical, symbol Connector_Generic:Conn_01x02
- added J13: BMS_OUT, Connector_PinHeader_2.54mm:PinHeader_1x02_P2.54mm_Vertical, symbol Connector_Generic:Conn_01x02
- added J35: AN0, Connector_PinHeader_2.54mm:PinHeader_1x02_P2.54mm_Vertical, symbol Connector_Generic:Conn_01x02
- C1: footprint (none) -> ElectricalProject:electrolytic capacitor
- D1: footprint (none) -> LED_THT:LED_D5.0mm
- J1, J2, J26, J27, J3, J31, J32, J33, J34: footprint (none) -> Connector_PinHeader_2.54mm:PinHeader_1x08_P2.54mm_Vertical
- J14, SW1, SW2, SW3: footprint (none) -> Connector_PinHeader_2.54mm:PinHeader_1x05_P2.54mm_Vertical
- J15, J17, J30: footprint (none) -> Connector_PinHeader_2.54mm:PinHeader_1x02_P2.54mm_Vertical
- J16, J24, J25, J9: footprint (none) -> Connector_PinHeader_2.54mm:PinHeader_1x06_P2.54mm_Vertical
- J18, J19: footprint (none) -> Connector_PinHeader_2.54mm:PinHeader_1x07_P2.54mm_Vertical
- J20, J23, J28: footprint (none) -> Connector_PinHeader_2.54mm:PinHeader_1x03_P2.54mm_Vertical
- J21, J22: footprint (none) -> Connector_PinHeader_2.54mm:PinHeader_1x04_P2.54mm_Vertical
- J29, J6: footprint (none) -> Connector_PinHeader_2.54mm:PinHeader_1x10_P2.54mm_Vertical
- J4: value Conn_01x08 -> PWM; footprint (none) -> Connector_PinHeader_2.54mm:PinHeader_1x08_P2.54mm_Vertical
- J5: value Conn_01x08 -> Comms; footprint (none) -> Connector_PinHeader_2.54mm:PinHeader_1x08_P2.54mm_Vertical
- J7: footprint (none) -> Connector_PinHeader_2.54mm:PinHeader_2x18_P2.54mm_Vertical
- J8: footprint (none) -> Connector:FanPinHeader_1x03_P2.54mm_Vertical
- R1, R10, R11, R12, R13, R14, R15, R16, R17, R18, R19, R2, R20, R21, R22, R23, R3, R4, R5, R6, R7, R8, R9: footprint (none) -> Resistor_THT:R_Axial_DIN0207_L6.3mm_D2.5mm_P5.08mm_Vertical
- SW4, SW5, SW6, SW7: footprint (none) -> Button_Switch_THT:SW_PUSH_6mm_H4.3mm
- U1: value LM741 -> LM833; footprint (none) -> Package_DIP:DIP-8_W7.62mm
- U2, U3, U4: footprint (none) -> Package_DIP:DIP-20_W7.62mm
Connections:
- net +5V: now also R12.2, R13.2, R14.2; no longer R12.1, R13.1, R14.1
- net D0: now also J4.8 (Pin_8)
- net D1: now also J4.7 (Pin_7)
- net D10: now also U2.11 (LE)
- net D2: now also J4.6 (Pin_6)
- net D22: no longer U2.3 (D0), U3.3 (D0), U4.3 (D0)
- net D23: no longer U2.13 (D4), U3.13 (D4), U4.13 (D4)
- net D24: no longer U2.4 (D1), U3.4 (D1), U4.4 (D1)
- net D25: no longer U2.14 (D5), U3.14 (D5), U4.14 (D5)
- net D26: no longer U2.7 (D2), U3.7 (D2), U4.7 (D2)
- net D27: no longer U2.17 (D6), U3.17 (D6), U4.17 (D6)
- net D28: no longer U2.8 (D3), U3.8 (D3), U4.8 (D3)
- net D29: no longer U2.18 (D7), U3.18 (D7), U4.18 (D7)
- net D3: now also J4.5 (Pin_5)
- net D30: now also U2.18 (D7), U3.18 (D7), U4.18 (D7); no longer R23.2, SW1.S1
- net D31: now also U2.17 (D6), U3.17 (D6), U4.17 (D6); no longer J24.2 (Pin_2)
- net D32: now also U2.14 (D5), U3.14 (D5), U4.14 (D5); no longer R7.2, SW1.A
- net D33: now also U2.13 (D4), U3.13 (D4), U4.13 (D4); no longer R14.2, SW1.B
- net D34: now also U2.8 (D3), U3.8 (D3), U4.8 (D3)
- net D35: now also U2.7 (D2), U3.7 (D2), U4.7 (D2)
- net D36: now also U2.4 (D1), U3.4 (D1), U4.4 (D1)
- net D37: now also U2.3 (D0), U3.3 (D0), U4.3 (D0)
- net D38: now also J24.2 (Pin_2)
- net D39: now also R14.1, SW3.3 (B)
- net D4: now also J4.4 (Pin_4), U3.11 (LE)
- net D40: now also R7.2, SW3.1 (A)
- net D41: now also R23.2, SW3.4 (S1)
- net D43: now also SW1.1 (A); no longer SW3.A
- net D44: now also R12.1, SW1.3 (B); no longer R12.2, SW3.B
- net D45: now also SW1.4 (S1); no longer SW3.S1
- net D47: now also R13.1, SW2.3 (B); no longer R13.2, SW2.B
- net D48: now also SW2.1 (A); no longer SW2.A
- net D49: now also SW2.4 (S1); no longer SW2.S1
- net D5: now also J4.3 (Pin_3)
- net D58: now also U4.11 (LE); no longer U2.1 (OE), U3.1 (OE), U4.1 (OE)
- net D6: now also J4.2 (Pin_2)
- net D64: no longer J26.5 (Pin_5), J3.5 (Pin_5)
- net D65: no longer J26.6 (Pin_6), J3.6 (Pin_6)
- net D66: now also J26.5 (Pin_5), J3.5 (Pin_5); no longer J26.7 (Pin_7), J3.7 (Pin_7)
- net D67: now also J26.6 (Pin_6), J3.6 (Pin_6); no longer J26.8 (Pin_8), J3.8 (Pin_8)
- net D7: now also J4.1 (Pin_1)
- net D9: now also U2.1 (OE), U3.1 (OE), U4.1 (OE); no longer U2.11 (LE), U3.11 (LE), U4.11 (LE)
- net GNDPWR: now also J8.3 (MountPin), SW1.2 (C), SW1.5 (S2), SW2.2 (C), SW2.5 (S2), SW3.2 (C), SW3.5 (S2), J10.2 (Pin_2), J11.2 (Pin_2), J12.2 (Pin_2), J13.1 (Pin_1), J35.2 (Pin_2); no longer J8.MP (MountPin), SW1.C, SW1.S2, SW2.C, SW2.S2, SW3.C, SW3.S2
- net at R18.1: now also J12.1 (Pin_1)
- net at R16.1: now also J10.1 (Pin_1)
- net at R15.1: now also J35.1 (Pin_1)
- net at R17.1: now also J11.1 (Pin_1)
- net S1 renamed +15V
- net +15V: now also J13.2 (Pin_2)
- new net D68: J26.7 (Pin_7), J3.7 (Pin_7)
- new net D69: J26.8 (Pin_8), J3.8 (Pin_8)
Other:
- moved on the sheet: C1, D1, D2, D3, D4, D5, J1, J14, J15, J16, J17, J18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
