File: ElectricalProject/ArduinoIHM.kicad_sch (KiCad schematic)
At the start: 76 parts, among them J1 PWR-CONNECTORS, J10 AN1, J11 AN2, J12 AN3, J13 BMS_OUT, J14 PWR, J15 DAC0_out, J16 DAC1, J17 DAC1_out, J18 Can0, J19 Can1, J2 PF 0 - 7, J20 RS485, J21 PWM0, J22 PWM1, J23 PWM2, J24 D-J3, J25 D-J4, J26 D-J2, J27 D-J1, J28 COMM, J29 Conn_01x10, J3 PK 8-15, J30 OrientationDet, J31 ServoSig, J32 VccLine, J33 GndLine, J34 DCMotorOut, J35 AN0, J4 PWM, J5 Comms, J6 PWM, J7 DigitalIO, J8 external_PWR, J9 DAC0, Q1 BC547, SW1 RotaryEncoder_Switch, SW2 RotaryEncoder_Switch, SW3 RotaryEncoder_Switch, SW4 SW_Push, SW5 SW_Push, SW6 SW_Push, SW7 SW_Push, U1 LM833, U2 74LS373, U3 74LS373, U4 74LS373

Commit message: Add architecture documentation; discover multiplexed output bus
Full documentation pass: ARCHITECTURE.md, a README in every lib/ module
and src/, and a drawio diagram covering the module map, scheduling
model, and known gaps.

While investigating a suspected Timer4 register conflict between PWM
channel 3 and a planned ServoMotor wiring, cross-checking against the
user's IOs IHM.xlsx and KiCad schematic revealed that Relay/ServoMotor/
MotorDC don't drive independent GPIO pins at all -- they share one 8-bit
bus behind three 74LS373 latches, addressed by per-device strobe lines
(dig_0/dig_1/dig_2). BinaryOutputs::SetOutput() doesn't implement this
protocol, so Relay's existing UI wiring likely doesn't work on real
hardware. This supersedes the original Timer4-conflict framing (moot --
ServoMotor never touches a PWM timer under this design) and is now
NEXT-SESSION.md's top priority.

Co-Authored-By: Claude Sonnet 5 <noreply@anthropic.com>
Parts:
- J29: value Conn_01x10 -> relays
Changed lines of the file:
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@@
 			)
 		)
-		(property "Value" "Conn_01x10"
+		(property "Value" "relays"
 			(at 271.526 53.848 0)
 			(effects
