File: ElectricalProject/ArduinoIHM.kicad_sch (KiCad schematic)
At the start: 76 parts, among them J1 PWR-CONNECTORS, J10 AN1, J11 AN2, J12 AN3, J13 BMS_OUT, J14 PWR, J15 DAC0_out, J16 DAC1, J17 DAC1_out, J18 Can0, J19 Can1, J2 PF 0 - 7, J20 RS485, J21 PWM0, J22 PWM1, J23 PWM2, J24 D-J3, J25 D-J4, J26 D-J2, J27 D-J1, J28 COMM, J29 relays, J3 PK 8-15, J30 OrientationDet, J31 ServoSig, J32 VccLine, J33 GndLine, J34 DCMotorOut, J35 AN0, J4 PWM, J5 Comms, J6 PWM, J7 DigitalIO, J8 external_PWR, J9 DAC0, Q1 BC547, SW1 RotaryEncoder_Switch, SW2 RotaryEncoder_Switch, SW3 RotaryEncoder_Switch, SW4 SW_Push, SW5 SW_Push, SW6 SW_Push, SW7 SW_Push, U1 LM833, U2 74LS373, U3 74LS373, U4 74LS373

Commit message: Sync IOs IHM.xlsx (v0) pin plan with ArduinoIHM.kicad_sch
Relabeled global_label pin numbers across the encoder/output-bus
region to match the "v0" sheet's new plan, and fixed a leftover
LCD_RST label that was still on D38 (shorted against rotary
encoder 2's channel-A switch) instead of its new D31 assignment.

Note: this is the last commit before the IO change.
Connections:
- net D10: no longer U2.11 (LE)
- net D30: now also R21.2, SW1.4 (S1); no longer U2.18 (D7), U3.18 (D7), U4.18 (D7)
- net D31: now also J24.2 (Pin_2); no longer U2.17 (D6), U3.17 (D6), U4.17 (D6)
- net D32: now also R12.1, SW1.3 (B); no longer U2.14 (D5), U3.14 (D5), U4.14 (D5)
- net D33: now also R4.2, SW1.1 (A); no longer U2.13 (D4), U3.13 (D4), U4.13 (D4)
- net D34: no longer U2.8 (D3), U3.8 (D3), U4.8 (D3)
- net D35: now also R7.2, SW3.1 (A); no longer U2.7 (D2), U3.7 (D2), U4.7 (D2)
- net D36: now also R14.1, SW3.3 (B); no longer U2.4 (D1), U3.4 (D1), U4.4 (D1)
- net D37: now also R23.2, SW3.4 (S1); no longer U2.3 (D0), U3.3 (D0), U4.3 (D0)
- net D38: now also R6.2, SW2.1 (A); no longer J24.2 (Pin_2)
- net D39: now also R13.1, SW2.3 (B); no longer R14.1, SW3.3 (B)
- net D40: now also R22.2, SW2.4 (S1); no longer R7.2, SW3.1 (A)
- net D41: now also U2.1 (OE), U3.1 (OE), U4.1 (OE); no longer R23.2, SW3.4 (S1)
- net D42: now also U2.18 (D7), U3.18 (D7), U4.18 (D7)
- net D43: now also U2.17 (D6), U3.17 (D6), U4.17 (D6); no longer R4.2, SW1.1 (A)
- net D44: now also U2.14 (D5), U3.14 (D5), U4.14 (D5); no longer R12.1, SW1.3 (B)
- net D45: now also U2.13 (D4), U3.13 (D4), U4.13 (D4); no longer R21.2, SW1.4 (S1)
- net D46: now also U2.8 (D3), U3.8 (D3), U4.8 (D3)
- net D47: now also U2.7 (D2), U3.7 (D2), U4.7 (D2); no longer R13.1, SW2.3 (B)
- net D48: now also U2.4 (D1), U3.4 (D1), U4.4 (D1); no longer R6.2, SW2.1 (A)
- net D49: now also U2.3 (D0), U3.3 (D0), U4.3 (D0); no longer R22.2, SW2.4 (S1)
- net D9: now also U2.11 (LE); no longer U2.1 (OE), U3.1 (OE), U4.1 (OE)
Changed lines of the file:
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@@
 		)
 	)
-	(global_label "D49"
+	(global_label "D40"
 		(shape bidirectional)
 		(at 77.47 52.07 0)
@@
 		)
 	)
-	(global_label "D43"
+	(global_label "D33"
 		(shape bidirectional)
 		(at 24.13 80.01 180)
@@
 		)
 	)
-	(global_label "D36"
+	(global_label "D48"
 		(shape bidirectional)
 		(at 220.98 120.65 180)
@@
 		)
 	)
-	(global_label "D47"
+	(global_label "D39"
 		(shape bidirectional)
 		(at 25.4 57.15 180)
@@
 		)
 	)
-	(global_label "D10"
+	(global_label "D9"
 		(shape bidirectional)
 		(at 240.03 53.34 180)
@@
 		)
 		(property "Intersheetrefs" "${INTERSHEET_REFS}"
-			(at 232.2445 53.34 0)
+			(at 233.454 53.34 0)
 			(effects
 				(font
@@
 		)
 	)
-	(global_label "D9"
+	(global_label "D41"
 		(shape bidirectional)
 		(at 238.76 101.6 180)
@@
 		)
 		(property "Intersheetrefs" "${INTERSHEET_REFS}"
-			(at 232.184 101.6 0)
+			(at 230.9745 101.6 0)
 			(effects
 				(font
@@
 		)
 	)
-	(global_label "D37"
+	(global_label "D49"
 		(shape bidirectional)
 		(at 220.98 118.11 180)
@@
 		)
 	)
-	(global_label "D39"
+	(global_label "D36"
 		(shape bidirectional)
 		(at 24.13 33.02 180)
@@
 		)
 	)
-	(global_label "D48"
+	(global_label "D38"
 		(shape bidirectional)
 		(at 25.4 52.07 180)
@@
 		)
 	)
-	(global_label "D32"
+	(global_label "D44"
 		(shape bidirectional)
 		(at 220.98 130.81 180)
@@
 		)
 	)
-	(global_label "D41"
+	(global_label "D37"
 		(shape bidirectional)
 		(at 74.93 27.94 0)
@@
 		)
 	)
-	(global_label "D31"
+	(global_label "D43"
 		(shape bidirectional)
 		(at 220.98 133.35 180)
@@
 		)
 	)
-	(global_label "D38"
+	(global_label "D31"
 		(shape input)
 		(at 138.43 147.32 0)
@@
 		)
 	)
-	(global_label "D30"
+	(global_label "D42"
 		(shape bidirectional)
 		(at 220.98 135.89 180)
@@
 		)
 	)
-	(global_label "D40"
+	(global_label "D35"
 		(shape bidirectional)
 		(at 24.13 27.94 180)
@@
 		)
 	)
-	(global_label "D45"
+	(global_label "D30"
 		(shape bidirectional)
 		(at 77.47 80.01 0)
@@
 		)
 	)
-	(global_label "D34"
+	(global_label "D46"
 		(shape bidirectional)
 		(at 220.98 125.73 180)
@@
 		)
 	)
-	(global_label "D33"
+	(global_label "D45"
 		(shape bidirectional)
 		(at 220.98 128.27 180)
@@
 		)
 	)
-	(global_label "D35"
+	(global_label "D47"
 		(shape bidirectional)
 		(at 220.98 123.19 180)
@@
 		)
 	)
-	(global_label "D44"
+	(global_label "D32"
 		(shape bidirectional)
 		(at 24.13 85.09 180)
@@
 		)
 	)
-	(global_label "D9"
+	(global_label "D41"
 		(shape bidirectional)
 		(at 238.76 147.32 180)
@@
 		)
 		(property "Intersheetrefs" "${INTERSHEET_REFS}"
-			(at 232.184 147.32 0)
+			(at 230.9745 147.32 0)
 			(effects
 				(font
@@
 		)
 	)
-	(global_label "D9"
+	(global_label "D41"
 		(shape bidirectional)
 		(at 240.03 55.88 180)
@@
 		)
 		(property "Intersheetrefs" "${INTERSHEET_REFS}"
-			(at 233.454 55.88 0)
+			(at 232.2445 55.88 0)
 			(effects
 				(font
