File: ElectricalProject/ArduinoIHM.kicad_pcb (KiCad board)
At the start: 2 copper layers, 0 parts

Commit message: Restore ArduinoIHM.kicad_pcb footprint placement
This was uncommitted work-in-progress (76 placed footprints) sitting
in the working tree since around 2026-01-17, never committed. It was
accidentally discarded by a git reset --hard run while working on an
unrelated firmware branch; recovered from the KiCad backup zip
ElectricalProject/ArduinoIHM-backups/ArduinoIHM-2026-01-17_143124.zip
(still on disk, untracked), which matches the placement state
observed earlier in the same session.

No routing yet -- this is placement-only, same as before.

Co-Authored-By: Claude Sonnet 5 <noreply@anthropic.com>
Parts:
- added C1: 1u, ElectricalProject:electrolytic capacitor, F.Cu at (23.2, 159.8)
- added D1: LED, LED_THT:LED_D5.0mm, F.Cu at (21.3, 167.9)
- added D2: 1N4732, Diode_THT:D_DO-41_SOD81_P10.16mm_Horizontal, F.Cu at (225.8, 44.2)
- added D3: 1N4732, Diode_THT:D_DO-41_SOD81_P10.16mm_Horizontal, F.Cu at (225.8, 48.4)
- added D4: 1N4732, Diode_THT:D_DO-41_SOD81_P10.16mm_Horizontal, F.Cu at (225.8, 52.7)
- added D5: 1N4732, Diode_THT:D_DO-41_SOD81_P10.16mm_Horizontal, F.Cu at (225.8, 56.9)
- added J1: PWR-CONNECTORS, Connector_PinHeader_2.54mm:PinHeader_1x08_P2.54mm_Vertical, F.Cu at (121.4, 103.5)
- added J10: AN1, Connector_PinHeader_2.54mm:PinHeader_1x02_P2.54mm_Vertical, F.Cu at (21.1, 116.3)
- added J11: AN2, Connector_PinHeader_2.54mm:PinHeader_1x02_P2.54mm_Vertical, F.Cu at (25.7, 116.3)
- added J12: AN3, Connector_PinHeader_2.54mm:PinHeader_1x02_P2.54mm_Vertical, F.Cu at (30.3, 116.3)
- added J13: BMS_OUT, Connector_PinHeader_2.54mm:PinHeader_1x02_P2.54mm_Vertical, F.Cu at (34.9, 116.3)
- added J14: PWR, Connector_PinHeader_2.54mm:PinHeader_1x05_P2.54mm_Vertical, F.Cu at (-59.8, 16.2)
- added J15: DAC0_out, Connector_PinHeader_2.54mm:PinHeader_1x02_P2.54mm_Vertical, F.Cu at (39.5, 116.3)
- added J16: DAC1, Connector_PinHeader_2.54mm:PinHeader_1x06_P2.54mm_Vertical, F.Cu at (45.4, 155.9)
- added J17: DAC1_out, Connector_PinHeader_2.54mm:PinHeader_1x02_P2.54mm_Vertical, F.Cu at (44.0, 116.3)
- added J18: Can0, Connector_PinHeader_2.54mm:PinHeader_1x07_P2.54mm_Vertical, F.Cu at (31.6, 155.9)
- added J19: Can1, Connector_PinHeader_2.54mm:PinHeader_1x07_P2.54mm_Vertical, F.Cu at (36.2, 155.9)
- added J2: PF 0 - 7, Connector_PinHeader_2.54mm:PinHeader_1x08_P2.54mm_Vertical, F.Cu at (96.5, 103.5)
- added J20: RS485, Connector_PinHeader_2.54mm:PinHeader_1x03_P2.54mm_Vertical, F.Cu at (-54.7, 39.5)
- added J21: PWM0, Connector_PinHeader_2.54mm:PinHeader_1x04_P2.54mm_Vertical, F.Cu at (-46.0, 31.0)
- added J22: PWM1, Connector_PinHeader_2.54mm:PinHeader_1x04_P2.54mm_Vertical, F.Cu at (-41.4, 31.0)
- added J23: PWM2, Connector_PinHeader_2.54mm:PinHeader_1x03_P2.54mm_Vertical, F.Cu at (-55.2, 31.0)
- added J24: D-J3, Connector_PinHeader_2.54mm:PinHeader_1x06_P2.54mm_Vertical, F.Cu at (50.0, 155.9)
- added J25: D-J4, Connector_PinHeader_2.54mm:PinHeader_1x06_P2.54mm_Vertical, F.Cu at (-55.2, 16.2)
- added J26: D-J2, Connector_PinHeader_2.54mm:PinHeader_1x08_P2.54mm_Vertical, F.Cu at (198.7, 44.3)
- added J27: D-J1, Connector_PinHeader_2.54mm:PinHeader_1x08_P2.54mm_Vertical, F.Cu at (203.3, 44.3)
- added J28: COMM, Connector_PinHeader_2.54mm:PinHeader_1x03_P2.54mm_Vertical, F.Cu at (-50.6, 31.0)
- added J29: Conn_01x10, Connector_PinHeader_2.54mm:PinHeader_1x10_P2.54mm_Vertical, F.Cu at (225.5, 119.2)
- added J3: PK 8-15, Connector_PinHeader_2.54mm:PinHeader_1x08_P2.54mm_Vertical, F.Cu at (71.9, 103.5)
- added J30: OrientationDet, Connector_PinHeader_2.54mm:PinHeader_1x02_P2.54mm_Vertical, F.Cu at (48.6, 116.3)
- added J31: ServoSig, Connector_PinHeader_2.54mm:PinHeader_1x08_P2.54mm_Vertical, F.Cu at (207.9, 44.3)
- added J32: VccLine, Connector_PinHeader_2.54mm:PinHeader_1x08_P2.54mm_Vertical, F.Cu at (212.5, 44.3)
- added J33: GndLine, Connector_PinHeader_2.54mm:PinHeader_1x08_P2.54mm_Vertical, F.Cu at (217.1, 44.3)
- added J34: DCMotorOut, Connector_PinHeader_2.54mm:PinHeader_1x08_P2.54mm_Vertical, F.Cu at (221.7, 44.3)
- added J35: AN0, Connector_PinHeader_2.54mm:PinHeader_1x02_P2.54mm_Vertical, F.Cu at (53.2, 116.3)
- added J4: PWM, Connector_PinHeader_2.54mm:PinHeader_1x08_P2.54mm_Vertical, F.Cu at (103.1, 53.0)
- added J5: Comms, Connector_PinHeader_2.54mm:PinHeader_1x08_P2.54mm_Vertical, F.Cu at (78.5, 53.0)
- added J6: PWM, Connector_PinHeader_2.54mm:PinHeader_1x10_P2.54mm_Vertical, F.Cu at (133.2, 53.0)
- added J7: DigitalIO, Connector_PinHeader_2.54mm:PinHeader_2x18_P2.54mm_Vertical, F.Cu at (48.3, 53.2)
- added J8: external_PWR, Connector:FanPinHeader_1x03_P2.54mm_Vertical, F.Cu at (244.5, 26.3)
- added J9: DAC0, Connector_PinHeader_2.54mm:PinHeader_1x06_P2.54mm_Vertical, F.Cu at (40.8, 155.9)
- added Q1: BC547, Package_TO_SOT_THT:TO-92_Inline, F.Cu at (219.3, 67.7)
- added R1: 1k, Resistor_THT:R_Axial_DIN0207_L6.3mm_D2.5mm_P5.08mm_Vertical, F.Cu at (31.4, 123.2)
- added R10: 1k, Resistor_THT:R_Axial_DIN0207_L6.3mm_D2.5mm_P5.08mm_Vertical, F.Cu at (40.0, 127.3)
- added R11: 1k, Resistor_THT:R_Axial_DIN0207_L6.3mm_D2.5mm_P5.08mm_Vertical, F.Cu at (40.0, 131.3)
- added R12: 1k, Resistor_THT:R_Axial_DIN0207_L6.3mm_D2.5mm_P5.08mm_Vertical, F.Cu at (40.0, 135.4)
- added R13: 1k, Resistor_THT:R_Axial_DIN0207_L6.3mm_D2.5mm_P5.08mm_Vertical, F.Cu at (40.0, 139.4)
- added R14: 1k, Resistor_THT:R_Axial_DIN0207_L6.3mm_D2.5mm_P5.08mm_Vertical, F.Cu at (40.0, 143.5)
- added R15: 10k, Resistor_THT:R_Axial_DIN0207_L6.3mm_D2.5mm_P5.08mm_Vertical, F.Cu at (40.0, 147.5)
- added R16: 10k, Resistor_THT:R_Axial_DIN0207_L6.3mm_D2.5mm_P5.08mm_Vertical, F.Cu at (40.0, 151.6)
- added R17: 10k, Resistor_THT:R_Axial_DIN0207_L6.3mm_D2.5mm_P5.08mm_Vertical, F.Cu at (48.7, 123.2)
- added R18: 10k, Resistor_THT:R_Axial_DIN0207_L6.3mm_D2.5mm_P5.08mm_Vertical, F.Cu at (48.7, 127.3)
- added R19: 5k7, Resistor_THT:R_Axial_DIN0207_L6.3mm_D2.5mm_P5.08mm_Vertical, F.Cu at (48.7, 131.3)
- added R2: 1K, Resistor_THT:R_Axial_DIN0207_L6.3mm_D2.5mm_P5.08mm_Vertical, F.Cu at (31.4, 127.3)
- added R20: 2k2, Resistor_THT:R_Axial_DIN0207_L6.3mm_D2.5mm_P5.08mm_Vertical, F.Cu at (48.7, 135.4)
- added R21: 1k, Resistor_THT:R_Axial_DIN0207_L6.3mm_D2.5mm_P5.08mm_Vertical, F.Cu at (48.7, 139.4)
- added R22: 1k, Resistor_THT:R_Axial_DIN0207_L6.3mm_D2.5mm_P5.08mm_Vertical, F.Cu at (48.7, 143.5)
- added R23: 1k, Resistor_THT:R_Axial_DIN0207_L6.3mm_D2.5mm_P5.08mm_Vertical, F.Cu at (48.7, 147.5)
- added R3: 0.01, Resistor_THT:R_Axial_DIN0207_L6.3mm_D2.5mm_P5.08mm_Vertical, F.Cu at (31.4, 131.3)
- added R4: 1k, Resistor_THT:R_Axial_DIN0207_L6.3mm_D2.5mm_P5.08mm_Vertical, F.Cu at (31.4, 135.4)
- added R5: 220, Resistor_THT:R_Axial_DIN0207_L6.3mm_D2.5mm_P5.08mm_Vertical, F.Cu at (31.4, 139.4)
- added R6: 1k, Resistor_THT:R_Axial_DIN0207_L6.3mm_D2.5mm_P5.08mm_Vertical, F.Cu at (31.4, 143.5)
- added R7: 1k, Resistor_THT:R_Axial_DIN0207_L6.3mm_D2.5mm_P5.08mm_Vertical, F.Cu at (31.4, 147.5)
- added R8: 1k, Resistor_THT:R_Axial_DIN0207_L6.3mm_D2.5mm_P5.08mm_Vertical, F.Cu at (31.4, 151.6)
- added R9: 1k, Resistor_THT:R_Axial_DIN0207_L6.3mm_D2.5mm_P5.08mm_Vertical, F.Cu at (40.0, 123.2)
- added SW1: RotaryEncoder_Switch, Connector_PinHeader_2.54mm:PinHeader_1x05_P2.54mm_Vertical, F.Cu at (-50.6, 16.2)
- added SW2: RotaryEncoder_Switch, Connector_PinHeader_2.54mm:PinHeader_1x05_P2.54mm_Vertical, F.Cu at (-46.0, 16.2)
- added SW3: RotaryEncoder_Switch, Connector_PinHeader_2.54mm:PinHeader_1x05_P2.54mm_Vertical, F.Cu at (-41.4, 16.2)
- added SW4: SW_Push, Button_Switch_THT:SW_PUSH_6mm_H4.3mm, F.Cu at (20.8, 123.2)
- added SW5: SW_Push, Button_Switch_THT:SW_PUSH_6mm_H4.3mm, F.Cu at (20.8, 131.8)
- added SW6: SW_Push, Button_Switch_THT:SW_PUSH_6mm_H4.3mm, F.Cu at (20.8, 140.3)
- added SW7: SW_Push, Button_Switch_THT:SW_PUSH_6mm_H4.3mm, F.Cu at (20.8, 148.9)
- added U1: LM833, Package_DIP:DIP-8_W7.62mm, F.Cu at (239.5, 44.1)
- added U2: 74LS373, Package_DIP:DIP-20_W7.62mm, F.Cu at (25.5, 83.9)
- added U3: 74LS373, Package_DIP:DIP-20_W7.62mm, F.Cu at (25.5, 52.9)
- added U4: 74LS373, Package_DIP:DIP-20_W7.62mm, F.Cu at (25.5, 20.8)
